Commit message: updated model.urdf

File: demo_pkg/urdf/model.urdf (robot description, URDF)
Before this commit: robot SingleMotorBot, 2 links, 1 joints
Links:
- removed link base_link
- removed link head
- added link spinning_box; visual box size=0.2 0.2 0.2
- added link stationary_base_link; visual cylinder length=0.6 radius=0.2
Joints:
- removed joint head_swivel
- added joint rotating_joint_1: type continuous, parent stationary_base_link, child spinning_box, origin xyz=0 0 0.3, axis 0 0 1
